File: PBSEQ-D2.kicad_sch (KiCad schematic)
At the start: 16 parts, among them J1 POWER IN, J2 POWER OUT, J3 BUTTON, Q1 AO3401A, Q2 AO3400A, SW1 BUTTON

Commit message: Updated resistor values
* Updated values of `R1` and `R4`. The new values are found to be working with practical testing.
* Updated `Q1` value to `AO3415` based on testing.
* Added net classes and highlights.
* Updated BoM.
* Imported new changes to the PCB.
* No changes in the electrical design.
Parts:
- Q1: value AO3401A -> AO3415; MPN AO3401A -> AO3415
- R4: value 100K -> 470K; MPN WR06X1003FTL -> WR06X4703FTL
Changed lines of the file:
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@@
 	(title_block
 		(title "PBSEQ-D2")
-		(date "2024-05-12")
+		(date "2024-08-01")
 		(rev "0.1")
 		(company "CIRCUITSTATE Electronics LLP")
@@
 		)
 	)
+	(netclass_flag ""
+		(length 2.54)
+		(shape round)
+		(at 90.805 85.725 0)
+		(effects
+			(font
+				(size 1.27 1.27)
+			)
+			(justify left bottom)
+		)
+		(property "Netclass" "GND"
+			(at 90.8685 81.915 0)
+			(effects
+				(font
+					(size 0.8 0.8)
+					(italic yes)
+				)
+			)
+		)
+	)
+	(netclass_flag ""
+		(length 2.54)
+		(shape round)
+		(at 71.12 52.07 0)
+		(effects
+			(font
+				(size 1.27 1.27)
+			)
+			(justify left bottom)
+		)
+		(property "Netclass" "VCC"
+			(at 71.1835 48.26 0)
+			(effects
+				(font
+					(size 0.8 0.8)
+					(italic yes)
+				)
+			)
+		)
+	)
 	(symbol
 		(lib_id "power:GND")
@@
 			)
 		)
-		(property "Value" "100K"
+		(property "Value" "470K"
 			(at 65.405 66.294 90)
 			(effects
@@
 			)
 		)
-		(property "MPN" "WR06X1003FTL"
+		(property "MPN" "WR06X4703FTL"
 			(at 65.405 64.77 0)
 			(effects
@@
 			)
 		)
-		(property "Value" "AO3401A"
+		(property "Value" "AO3415"
 			(at 82.55 47.752 90)
 			(effects
@@
 			)
 		)
-		(property "MPN" "AO3401A"
+		(property "MPN" "AO3415"
 			(at 82.55 54.61 0)
 			(effects
